File: BikeComputer.kicad_pcb (KiCad board)
At the start: 2 copper layers, 45.7 x 48.3 mm, 29 parts, among them IC1 ATMEGA328-P, P1 Serial, P2 OLED screen, SW1 SW_PUSH, SW2 SW_PUSH, SW3 SW_PUSH, U1 7805, U2 ISP, U3 LP298X, U4 4050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

Commit message: Changed to use the TQFP version of the 328P
Added a battery connector

Moved over to use 3.3v only as all bar the hall sensor are 3.3v capable. TODO find a replacement hall sensor that is 3.3v.
Parts:
- removed C1, C3: 10uF, Capacitors_SMD:c_elec_6.3x4.5
- removed U1: 7805, Power_Integrations:TO-220
- removed U4: 4050, SMD_Packages:SSOP-14
- added P3: Batt, Pin_Headers:Pin_Header_Straight_1x02, F.Cu at (184.0, 96.0)
- IC1: footprint Housings_DIP:DIP-28_W7.62mm -> Housings_QFP:TQFP-32_7x7mm_Pitch0.8mm
- P2: footprint Pin_Headers:Pin_Header_Straight_1x07 -> Socket_Strips:Socket_Strip_Straight_1x07
- moved C2 187.8 mm to (234.0, 91.0)
- moved C4 187.8 mm to (234.0, 99.0)
- moved C5 187.8 mm to (234.0, 95.0)
- moved C6 187.8 mm to (234.0, 104.0)
- moved C7 187.8 mm to (234.0, 108.0)
- moved C8 187.8 mm to (239.0, 91.0)
- moved C9 187.8 mm to (239.0, 95.0)
- moved D1 187.8 mm to (262.0, 63.0)
- moved D2 187.8 mm to (263.0, 67.0)
- moved P1 187.8 mm to (239.0, 56.0)
- moved R1 187.8 mm to (205.0, 68.0)
- moved R2 187.8 mm to (205.0, 73.0)
- moved R3 187.8 mm to (205.0, 77.0)
- moved R4 187.8 mm to (205.0, 82.0)
- moved R5 187.8 mm to (205.0, 86.0)
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Connections:
- C6 pad 1: +5V -> +BATT
- C8 pad 1: +5V -> +3V3
- D2 pad 2: Net-(D2-Pad2) -> /SCK
- IC1 pad 1: /Reset -> (no net)
- IC1 pad 10: Net-(C5-Pad2) -> /Button_Select
- IC1 pad 11: /Button_Down -> Net-(D1-Pad2)
- IC1 pad 12: /Button_Select -> (no net)
- IC1 pad 13: Net-(D1-Pad2) -> /SD_Select
- IC1 pad 14: (no net) -> /Screen_Select
- IC1 pad 15: /SD_Select -> /MOSI
- IC1 pad 16: /Screen_Select -> /MISO
- IC1 pad 17: /MOSI -> /SCK
- IC1 pad 18: /MISO -> +3V3
- IC1 pad 19: /SCK -> (no net)
- IC1 pad 2: /Rx -> /Button_Up
- IC1 pad 20: +5V -> Net-(C9-Pad1)
- IC1 pad 21: Net-(C9-Pad1) -> GND
- IC1 pad 22: GND -> (no net)
- IC1 pad 3: /Tx -> GND
- IC1 pad 4: /Hall -> +3V3
- IC1 pad 5: (no net) -> GND
- IC1 pad 6: /Button_Up -> +3V3
- IC1 pad 7: +5V -> Net-(C4-Pad2)
- IC1 pad 8: GND -> Net-(C5-Pad2)
- IC1 pad 9: Net-(C4-Pad2) -> /Button_Down
- P1 pad 3: +5V -> +3V3
- P2 pad 2: +5V -> +3V3
- R1 pad 1: +5V -> +3V3
- R2 pad 1: +5V -> +3V3
- R3 pad 1: +5V -> +3V3
- R5 pad 1: +5V -> +3V3
- R6 pad 1: Net-(J1-Pad2) -> /SD_Select
- U2 pad 2: +5V -> +3V3
- U3 pad 1: +5V -> +BATT
- U3 pad 3: +5V -> +BATT
- U5 pad 1: +5V -> +3V3
Routing:
- net /MOSI: track 16.8 -> 0.00 mm
- net /Screen_Select: track 11.7 -> 0.00 mm
- net /SCK: track 11.7 -> 0.00 mm
- net +5V: track 11.7 -> 0.00 mm
