File: BikeComputer.sch (KiCad schematic (older format))
At the start: 30 parts, among them IC1 ATMEGA328-P, J1 MICRO_SD_HINGE, P1 Serial, P2 OLED screen, SW1 SW_PUSH, SW2 SW_PUSH, SW3 SW_PUSH, U1 7805, U2 ISP, U3 LP298X, U4 4050, U5 A3144, Y1 Crystal 16MHz

Commit message: Assigned footprints and started on PCB
Parts:
- C1, C3: footprint (none) -> Capacitors_SMD:c_elec_6.3x4.5
- C2, C4, C5, C6, C7: footprint (none) -> Capacitors_SMD:C_0603_HandSoldering
- C8, C9: value 0.1p -> 0.1uF; footprint (none) -> Capacitors_SMD:C_0603_HandSoldering
- D1, D2: footprint (none) -> LEDs:LED_0603
- IC1: footprint DIL28 -> Housings_DIP:DIP-28_W7.62mm
- P1: footprint (none) -> Pin_Headers:Pin_Header_Straight_1x06
- P2: footprint (none) -> Pin_Headers:Pin_Header_Straight_1x07
- R1, R2, R3, R4, R5, R6: footprint (none) -> Resistors_SMD:R_0603_HandSoldering
- SW1, SW2, SW3: footprint (none) -> Buttons_Switches_ThroughHole:SW_PUSH
- U1: footprint (none) -> Power_Integrations:TO-220
- U2: footprint (none) -> Pin_Headers:Pin_Header_Straight_2x03
- U3: footprint (none) -> TO_SOT_Packages_SMD:SOT-23-5
- U4: footprint (none) -> SMD_Packages:SSOP-14
- U5: footprint (none) -> Pin_Headers:Pin_Header_Straight_1x03
- Y1: footprint (none) -> Crystals:Crystal_HC50-U_Vertical
Changed lines of the file:
@@
 LIBS:contrib
 LIBS:valves
-LIBS:BikeComputer
 LIBS:BikeComputer-cache
 EELAYER 25 0
@@
 F 0 "IC1" H 4100 3500 50  0000 L BNN
 F 1 "ATMEGA328-P" H 5250 850 50  0000 L BNN
-F 2 "DIL28" H 4850 2250 50  0000 C CIN
+F 2 "Housings_DIP:DIP-28_W7.62mm" H 4850 2250 50  0000 C CIN
 F 3 "" H 4850 2250 50  0000 C CNN
 	1    4850 2250
@@
 F 0 "Y1" V 6900 1800 50  0000 C CNN
 F 1 "Crystal 16MHz" V 6300 1800 50  0000 C CNN
-F 2 "" H 6600 1800 50  0000 C CNN
+F 2 "Crystals:Crystal_HC50-U_Vertical" H 6600 1800 50  0001 C CNN
 F 3 "" H 6600 1800 50  0000 C CNN
 	1    6600 1800
@@
 F 0 "C4" V 7000 1550 50  0000 L CNN
 F 1 "22pF" V 7300 1550 50  0000 L CNN
-F 2 "" H 7188 1450 50  0000 C CNN
+F 2 "Capacitors_SMD:C_0603_HandSoldering" H 7188 1450 50  0001 C CNN
 F 3 "" H 7150 1600 50  0000 C CNN
 	1    7150 1600
@@
 F 0 "C5" V 7000 1950 50  0000 L CNN
 F 1 "22pF" V 7300 1950 50  0000 L CNN
-F 2 "" H 7188 1850 50  0000 C CNN
+F 2 "Capacitors_SMD:C_0603_HandSoldering" H 7188 1850 50  0001 C CNN
 F 3 "" H 7150 2000 50  0000 C CNN
 	1    7150 2000
@@
 F 0 "U1" H 1700 854 50  0000 C CNN
 F 1 "7805" H 1550 1250 50  0000 C CNN
-F 2 "" H 1550 1050 50  0000 C CNN
+F 2 "Power_Integrations:TO-220" H 1550 1050 50  0001 C CNN
 F 3 "" H 1550 1050 50  0000 C CNN
 	1    1550 1050
@@
 F 0 "C1" H 925 1400 50  0000 L CNN
 F 1 "10uF" H 925 1200 50  0000 L CNN
-F 2 "" H 938 1150 50  0000 C CNN
+F 2 "Capacitors_SMD:c_elec_6.3x4.5" H 938 1150 50  0001 C CNN
 F 3 "" H 900 1300 50  0000 C CNN
 	1    900  1300
@@
 F 0 "C3" H 2175 1400 50  0000 L CNN
 F 1 "10uF" H 2175 1200 50  0000 L CNN
-F 2 "" H 2188 1150 50  0000 C CNN
+F 2 "Capacitors_SMD:c_elec_6.3x4.5" H 2188 1150 50  0001 C CNN
 F 3 "" H 2150 1300 50  0000 C CNN
 	1    2150 1300
@@
 F 0 "U2" H 1650 5000 60  0000 C CNN
 F 1 "ISP" H 1650 5500 60  0000 C CNN
-F 2 "" H 1650 5250 60  0001 C CNN
+F 2 "Pin_Headers:Pin_Header_Straight_2x03" H 1650 5250 60  0001 C CNN
 F 3 "" H 1650 5250 60  0001 C CNN
 	1    1650 5250
@@
 F 0 "P1" H 1350 6400 50  0000 C CNN
 F 1 "Serial" V 1450 6050 50  0000 C CNN
-F 2 "" H 1350 6050 50  0000 C CNN
+F 2 "Pin_Headers:Pin_Header_Straight_1x06" H 1350 6050 50  0001 C CNN
 F 3 "" H 1350 6050 50  0000 C CNN
 	1    1350 6050
@@
 F 0 "C2" H 2025 5900 50  0000 L CNN
 F 1 "C" H 2025 5700 50  0000 L CNN
-F 2 "" H 2038 5650 50  0000 C CNN
+F 2 "Capacitors_SMD:C_0603_HandSoldering" H 2038 5650 50  0001 C CNN
 F 3 "" H 2000 5800 50  0000 C CNN
 	1    2000 5800
@@
 F 0 "D1" H 5950 3750 50  0000 C CNN
 F 1 "LED" H 5950 3550 50  0000 C CNN
-F 2 "" H 5950 3650 50  0000 C CNN
+F 2 "LEDs:LED_0603" H 5950 3650 50  0001 C CNN
 F 3 "" H 5950 3650 50  0000 C CNN
 	1    5950 3650
@@
 F 0 "R4" V 6030 4050 50  0000 C CNN
 F 1 "R" V 5950 4050 50  0000 C CNN
-F 2 "" V 5880 4050 50  0000 C CNN
+F 2 "Resistors_SMD:R_0603_HandSoldering" V 5880 4050 50  0001 C CNN
 F 3 "" H 5950 4050 50  0000 C CNN
 	1    5950 4050
@@
 F 0 "U5" H 10050 1400 60  0000 C CNN
 F 1 "A3144" H 10050 1250 60  0000 C CNN
-F 2 "" H 10050 1000 60  0001 C CNN
+F 2 "Pin_Headers:Pin_Header_Straight_1x03" H 10050 1000 60  0001 C CNN
 F 3 "" H 10050 1000 60  0001 C CNN
 	1    10050 1100
@@
 F 0 "R5" V 10480 1600 50  0000 C CNN
 F 1 "10K" V 10400 1600 50  0000 C CNN
-F 2 "" V 10330 1600 50  0000 C CNN
+F 2 "Resistors_SMD:R_0603_HandSoldering" V 10330 1600 50  0001 C CNN
 F 3 "" H 10400 1600 50  0000 C CNN
 	1    10400 1600
@@
 F 0 "P2" H 1350 7500 50  0000 C CNN
 F 1 "OLED screen" V 1450 7100 50  0000 C CNN
-F 2 "" H 1350 7100 50  0000 C CNN
+F 2 "Pin_Headers:Pin_Header_Straight_1x07" H 1350 7100 50  0001 C CNN
 F 3 "" H 1350 7100 50  0000 C CNN
 	1    1350 7100
@@
 F 0 "U4" H 8345 3615 50  0000 C CNN
 F 1 "4050" H 8340 3375 50  0000 C CNN
-F 2 "" H 8150 3500 60  0001 C CNN
+F 2 "SMD_Packages:SSOP-14" H 8150 3500 60  0001 C CNN
 F 3 "" H 8150 3500 60  0001 C CNN
 	1    8150 3500
@@
 F 0 "U4" H 8345 3965 50  0000 C CNN
 F 1 "4050" H 8340 3725 50  0000 C CNN
-F 2 "" H 8150 3850 60  0001 C CNN
+F 2 "SMD_Packages:SSOP-14" H 8150 3850 60  0001 C CNN
 F 3 "" H 8150 3850 60  0001 C CNN
 	2    8150 3850
@@
 F 0 "U4" H 8345 4315 50  0000 C CNN
 F 1 "4050" H 8340 4075 50  0000 C CNN
-F 2 "" H 8150 4200 60  0001 C CNN
+F 2 "SMD_Packages:SSOP-14" H 8150 4200 60  0001 C CNN
 F 3 "" H 8150 4200 60  0001 C CNN
 	3    8150 4200
@@
 F 0 "U4" H 8995 6015 50  0000 C CNN
 F 1 "4050" H 8990 5775 50  0000 C CNN
-F 2 "" H 8800 5900 60  0001 C CNN
+F 2 "SMD_Packages:SSOP-14" H 8800 5900 60  0001 C CNN
 F 3 "" H 8800 5900 60  0001 C CNN
 	5    8800 5900
@@
 F 0 "U4" H 9495 5365 50  0000 C CNN
 F 1 "4050" H 9490 5125 50  0000 C CNN
-F 2 "" H 9300 5250 60  0001 C CNN
+F 2 "SMD_Packages:SSOP-14" H 9300 5250 60  0001 C CNN
 F 3 "" H 9300 5250 60  0001 C CNN
 	4    9300 5250
@@
 F 0 "U4" H 10245 6015 50  0000 C CNN
 F 1 "4050" H 10240 5775 50  0000 C CNN
-F 2 "" H 10050 5900 60  0001 C CNN
+F 2 "SMD_Packages:SSOP-14" H 10050 5900 60  0001 C CNN
 F 3 "" H 10050 5900 60  0001 C CNN
 	6    10050 5900
@@
 F 0 "D2" H 10900 4500 50  0000 C CNN
 F 1 "LED" H 10900 4300 50  0000 C CNN
-F 2 "" H 10900 4400 50  0000 C CNN
+F 2 "LEDs:LED_0603" H 10900 4400 50  0001 C CNN
 F 3 "" H 10900 4400 50  0000 C CNN
 	1    10900 4400
@@
 F 0 "R6" V 10980 3700 50  0000 C CNN
 F 1 "R" V 10900 3700 50  0000 C CNN
-F 2 "" V 10830 3700 50  0000 C CNN
+F 2 "Resistors_SMD:R_0603_HandSoldering" V 10830 3700 50  0001 C CNN
 F 3 "" H 10900 3700 50  0000 C CNN
 	1    10900 3700
@@
 F 0 "C6" H 675 2650 50  0000 L CNN
 F 1 "C" H 675 2450 50  0000 L CNN
-F 2 "" H 688 2400 50  0000 C CNN
+F 2 "Capacitors_SMD:C_0603_HandSoldering" H 688 2400 50  0001 C CNN
 F 3 "" H 650 2550 50  0000 C CNN
 	1    650  2550
@@
 F 0 "C7" H 2675 2650 50  0000 L CNN
 F 1 "C" H 2675 2450 50  0000 L CNN
-F 2 "" H 2688 2400 50  0000 C CNN
+F 2 "Capacitors_SMD:C_0603_HandSoldering" H 2688 2400 50  0001 C CNN
 F 3 "" H 2650 2550 50  0000 C CNN
 	1    2650 2550
@@
 F 0 "U3" H 1950 1950 50  0000 C CNN
 F 1 "LP298X" H 1750 2850 50  0000 C CNN
-F 2 "" H 1750 2400 50  0000 C CNN
+F 2 "TO_SOT_Packages_SMD:SOT-23-5" H 1750 2400 50  0001 C CNN
 F 3 "" H 1750 2400 50  0000 C CNN
 	1    1750 2400
@@
 F 0 "J1" H 10200 4100 60  0000 C CNN
 F 1 "MICRO_SD_HINGE" H 10150 4600 60  0000 C CNN
-F 2 "" V 10260 3550 60  0000 C CNN
+F 2 "" V 10260 3550 60  0001 C CNN
 F 3 "" V 10260 3550 60  0000 C CNN
 	1    10150 4050
@@
 F 0 "SW1" H 4600 5860 50  0000 C CNN
 F 1 "SW_PUSH" H 4450 5670 50  0000 C CNN
-F 2 "" H 4450 5750 50  0000 C CNN
+F 2 "Buttons_Switches_ThroughHole:SW_PUSH" H 4450 5750 50  0001 C CNN
 F 3 "" H 4450 5750 50  0000 C CNN
 	1    4450 5750
@@
 F 0 "SW2" H 4600 6160 50  0000 C CNN
 F 1 "SW_PUSH" H 4450 5970 50  0000 C CNN
-F 2 "" H 4450 6050 50  0000 C CNN
+F 2 "Buttons_Switches_ThroughHole:SW_PUSH" H 4450 6050 50  0001 C CNN
 F 3 "" H 4450 6050 50  0000 C CNN
 	1    4450 6050
@@
 F 0 "SW3" H 4600 6460 50  0000 C CNN
 F 1 "SW_PUSH" H 4450 6270 50  0000 C CNN
-F 2 "" H 4450 6350 50  0000 C CNN
+F 2 "Buttons_Switches_ThroughHole:SW_PUSH" H 4450 6350 50  0001 C CNN
 F 3 "" H 4450 6350 50  0000 C CNN
 	1    4450 6350
@@
 F 0 "R3" V 5180 6350 50  0000 C CNN
 F 1 "R" V 5100 6350 50  0000 C CNN
-F 2 "" V 5030 6350 50  0000 C CNN
+F 2 "Resistors_SMD:R_0603_HandSoldering" V 5030 6350 50  0001 C CNN
 F 3 "" H 5100 6350 50  0000 C CNN
 	1    5100 6350
@@
 F 0 "R2" V 5180 6050 50  0000 C CNN
 F 1 "R" V 5100 6050 50  0000 C CNN
-F 2 "" V 5030 6050 50  0000 C CNN
+F 2 "Resistors_SMD:R_0603_HandSoldering" V 5030 6050 50  0001 C CNN
 F 3 "" H 5100 6050 50  0000 C CNN
 	1    5100 6050
@@
 F 0 "R1" V 5180 5750 50  0000 C CNN
 F 1 "R" V 5100 5750 50  0000 C CNN
-F 2 "" V 5030 5750 50  0000 C CNN
+F 2 "Resistors_SMD:R_0603_HandSoldering" V 5030 5750 50  0001 C CNN
 F 3 "" H 5100 5750 50  0000 C CNN
 	1    5100 5750
@@
 P 3350 2000
 F 0 "C8" H 3375 2100 50  0000 L CNN
-F 1 "0.1p" H 3375 1900 50  0000 L CNN
-F 2 "" H 3388 1850 50  0000 C CNN
+F 1 "0.1uF" H 3375 1900 50  0000 L CNN
+F 2 "Capacitors_SMD:C_0603_HandSoldering" H 3388 1850 50  0001 C CNN
 F 3 "" H 3350 2000 50  0000 C CNN
 	1    3350 2000
@@
 P 3700 2000
 F 0 "C9" H 3725 2100 50  0000 L CNN
-F 1 "0.1p" H 3725 1900 50  0000 L CNN
-F 2 "" H 3738 1850 50  0000 C CNN
+F 1 "0.1uF" H 3725 1900 50  0000 L CNN
+F 2 "Capacitors_SMD:C_0603_HandSoldering" H 3738 1850 50  0001 C CNN
 F 3 "" H 3700 2000 50  0000 C CNN
 	1    3700 2000

Commit message: Changed to use the TQFP version of the 328P
Added a battery connector

Moved over to use 3.3v only as all bar the hall sensor are 3.3v capable. TODO find a replacement hall sensor that is 3.3v.
Parts:
- removed C1, C3: 10uF, Capacitors_SMD:c_elec_6.3x4.5, symbol CP
- removed U1: 7805, Power_Integrations:TO-220, symbol 7805
- removed U4: 4050, SMD_Packages:SSOP-14, symbol 4050
- added P3: Batt, Pin_Headers:Pin_Header_Straight_1x02, symbol CONN_01X02
- IC1: footprint Housings_DIP:DIP-28_W7.62mm -> Housings_QFP:TQFP-32_7x7mm_Pitch0.8mm; symbol ATMEGA328-P -> ATMEGA328P-A
- P2: footprint Pin_Headers:Pin_Header_Straight_1x07 -> Socket_Strips:Socket_Strip_Straight_1x07
Connections:
- net +3V3: now also C8.1, IC1.18 (AVCC), IC1.4 (VCC), IC1.6 (VCC), P1.3 (P3), P2.2 (P2), R1.1, R2.1, R3.1, R5.1, U2.2 (Vcc), U5.1 (Vcc)
- net Button_Down: now also IC1.9 ((PCINT21/OC0B/T1)PD5); no longer IC1.11 ((PCINT21/OC0B/T1)PD5)
- net Button_Select: now also IC1.10 ((PCINT22/OC0A/AIN0)PD6); no longer IC1.12 ((PCINT22/OC0A/AIN0)PD6)
- net Button_Up: now also IC1.2 ((PCINT20/XCK/T0)PD4); no longer IC1.6 ((PCINT20/XCK/T0)PD4)
- net GND: now also IC1.21 (GND), IC1.3 (GND), IC1.5 (GND), P3.1 (P1); no longer IC1.22 (GND), IC1.8 (GND)
- net Hall: now also IC1.32 ((PCINT18/INT0)PD2); no longer IC1.4 ((PCINT18/INT0)PD2)
- net MISO: now also IC1.16 ((PCINT4/MISO)PB4); no longer IC1.18 ((PCINT4/MISO)PB4)
- net MOSI: now also IC1.15 ((PCINT3/OC2A/MOSI)PB3), J1.3 (CMD); no longer IC1.17 ((PCINT3/OC2A/MOSI)PB3)
- net Reset: now also IC1.29 ((PCINT14/~RESET~)PC6); no longer IC1.1 ((PCINT14/~RESET~)PC6)
- net Rx: now also IC1.30 ((PCINT16/RXD)PD0); no longer IC1.2 ((PCINT16/RXD)PD0)
- net SCK: now also D2.2 (A), IC1.17 ((PCINT5/SCK)PB5), J1.5 (CLK); no longer IC1.19 ((PCINT5/SCK)PB5)
- net SD_Select: now also IC1.13 ((PCINT1/OC1A)PB1), J1.2 (CD/DAT3), R6.1; no longer IC1.15 ((PCINT1/OC1A)PB1)
- net Screen_Select: now also IC1.14 ((PCINT2/OC1B/~SS~)PB2); no longer IC1.16 ((PCINT2/OC1B/~SS~)PB2)
- net Tx: now also IC1.31 ((PCINT17/TXD)PD1); no longer IC1.3 ((PCINT17/TXD)PD1)
- net at C5.2, Y1.1: now also IC1.8 ((PCINT7/XTAL2/TOSC2)PB7); no longer IC1.10 ((PCINT7/XTAL2/TOSC2)PB7)
- net at D1.2 (A): now also IC1.11 ((PCINT23/AIN1)PD7); no longer IC1.13 ((PCINT23/AIN1)PD7)
- net at C9.1: now also IC1.20 (AREF); no longer IC1.21 (AREF)
- net at C4.2, Y1.2: now also IC1.7 ((PCINT6/XTAL1/TOSC1)PB6); no longer IC1.9 ((PCINT6/XTAL1/TOSC1)PB6)
- removed net +5V: C6.1, C8.1, IC1.20 (AVCC), IC1.7 (VCC), P1.3 (P3), P2.2 (P2), R1.1, R2.1, R3.1, R5.1, U2.2 (Vcc), U3.1 (VIN), U3.3 (ON/OFF), U5.1 (Vcc)
- new net +BATT: C6.1, P3.2 (P2), U3.1 (VIN), U3.3 (ON/OFF)
Other:
- moved on the sheet: C2, C6, C7, P1, U2, U3
